Commit message: InitVesion

File: src/scorpio/scorpio_description/urdf/_d435.urdf.xacro (robot description, xacro)
@@ -43,5 +43,5 @@
     <link name="camera_link">
       <visual>
-      <origin xyz="${d435_cam_mount_from_center_offset} ${-d435_cam_depth_py} 0" rpy="${M_PI/2} 0 ${M_PI/2}"/>
+      <origin xyz="${d435_cam_mount_from_center_offset} ${-d435_cam_depth_py} -0.02" rpy="${M_PI/2} 0 ${M_PI/2}"/>
         <geometry>
           <!-- <box size="${d435_cam_width} ${d435_cam_height} ${d435_cam_depth}"/> -->

File: src/scorpio/scorpio_description/urdf/scorpio_red.urdf.xacro (robot description, xacro)
@@ -6,5 +6,5 @@
 -->
 <robot name="scorpio" xmlns:xacro="http://ros.org/wiki/xacro">
-  	<xacro:include filename="$(find scorpio_description)/urdf/base/car_base.urdf"/>
+  	<xacro:include filename="$(find scorpio_description)/urdf/base/car_base_red.urdf"/>
 	<!--<xacro:include filename="$(find scorpio_description)/urdf/sensors/lidar.urdf"/>-->
 	<xacro:include filename="$(find scorpio_description)/urdf/sensors/astra_camera.urdf" />

File: src/scorpio/scorpio_description/urdf/scorpio_silver.urdf.xacro (robot description, xacro)
@@ -6,5 +6,5 @@
 -->
 <robot name="scorpio" xmlns:xacro="http://ros.org/wiki/xacro">
-  	<xacro:include filename="$(find scorpio_description)/urdf/base/car_base.urdf"/>
+  	<xacro:include filename="$(find scorpio_description)/urdf/base/car_base_silver.urdf"/>
 	<xacro:include filename="$(find ydlidar_g2)/urdf/ydlidar.urdf" />
 	<xacro:include filename="$(find scorpio_description)/urdf/_d435.urdf.xacro" />
